Commit message: Added basic navstack with nav2 and rtabmap

File: unitree_go2_description/urdf/realsense_d435.xacro (robot description, xacro)
@@ -1,13 +1,13 @@
 <?xml version="1.0"?>
 <robot xmlns:xacro="http://www.ros.org/wiki/xacro">
-    <!-- Include the RealSense D455 URDF macro from realsense2_description -->
-    <xacro:include filename="$(find realsense2_description)/urdf/_d455.urdf.xacro"/>
-    <!-- Mount the D455 on top of the trunk, in front of the velodyne lidar -->
-    <xacro:sensor_d455 parent="trunk" name="d455_camera" use_nominal_extrinsics="true">
-        <origin xyz="0.28 0 0.062" rpy="0 0 0"/>
-    </xacro:sensor_d455>
+    <!-- Include the RealSense d435 URDF macro from realsense2_description -->
+    <xacro:include filename="$(find realsense2_description)/urdf/_d435.urdf.xacro"/>
+    <!-- Mount the d435 on top of the trunk, in front of the velodyne lidar -->
+    <xacro:sensor_d435 parent="trunk" name="d435_camera" use_nominal_extrinsics="true">
+        <origin xyz="0.28 0 0.07" rpy="0 0 0"/>
+    </xacro:sensor_d435>
     <!-- Gazebo Sim RGBD Camera sensor plugin -->
-    <gazebo reference="d455_camera_link">
-        <sensor name="d455_rgbd_camera" type="rgbd_camera">
+    <gazebo reference="d435_camera_link">
+        <sensor name="d435_rgbd_camera" type="rgbd_camera">
             <pose>0 0 0 0 0 0</pose>
             <camera>
@@ -25,6 +25,6 @@
             <update_rate>15</update_rate>
             <visualize>true</visualize>
-            <topic>d455</topic>
-            <gz_frame_id>d455_camera_link</gz_frame_id>
+            <topic>d435</topic>
+            <gz_frame_id>d435_camera_color_optical_frame</gz_frame_id>
         </sensor>
     </gazebo>

File: unitree_go2_description/urdf/unitree_go2_robot.xacro (robot description, xacro)
@@ -12,5 +12,5 @@
     <xacro:include filename="$(find unitree_go2_description)/urdf/velodyne.xacro"/>
     <xacro:include filename="$(find unitree_go2_description)/urdf/lidar_4D_lidar.xacro"/>
-    <xacro:include filename="$(find unitree_go2_description)/urdf/realsense_d455.xacro"/>
+    <xacro:include filename="$(find unitree_go2_description)/urdf/realsense_d435.xacro"/>
     <!-- <xacro:stairs stairs="15" xpos="0" ypos="0" zpos="0" /> -->
     <xacro:unitree_go2_gazebo robot_controllers="$(arg robot_controllers)"/>

File: unitree_go2_description/urdf/velodyne.xacro (robot description, xacro)
@@ -61,9 +61,15 @@
                         <max_angle>3.14159</max_angle>
                     </horizontal>
-                    <vertical>
+                    <!-- <vertical>
                         <samples>16</samples>
                         <resolution>1</resolution>
                         <min_angle>-0.261799</min_angle>
                         <max_angle>0.261799</max_angle>
+                    </vertical> -->
+                    <vertical>
+                        <samples>32</samples>
+                        <resolution>1</resolution>
+                        <min_angle>-0.523599</min_angle>   <!-- -30 deg -->
+                        <max_angle>0.261799</max_angle>    <!-- +15 deg -->
                     </vertical>
                 </scan>
